File: openchess-redesign/hardware-nodemcu/openchess-board-nodemcu.kicad_pcb (KiCad board)
At the start: 2 copper layers, 340 x 388 mm, 239 parts, among them J1 USB-C, J2 5V IN, J3 DEV_TOP, J4 DEV_BOTTOM, Q1 S8550, Q2 S8550, Q3 S8550, Q4 S8550, Q5 S8550, Q6 S8550, Q7 S8550, Q8 S8550, U4 74HCT595, U5 74AHCT1G125

Commit message: nodemcu: pre-route GND stubs for the socket GND pins
Co-Authored-By: Claude Fable 5.1 <noreply@anthropic.com>
Claude-Session: https://claude.ai/code/session_01BYqUw5RUauFb8joYQgSgKZ
Routing:
- net GND: track 0.00 -> 9.00 mm, vias 381 -> 384

Commit message: Pre-route 74HCT595 OE ground via; router margin 0.02 mm; GND repair adds pad stubs
Co-Authored-By: Claude Fable 5.1 <noreply@anthropic.com>
Claude-Session: https://claude.ai/code/session_01BYqUw5RUauFb8joYQgSgKZ
Routing:
- net GND: track 9.00 -> 11.6 mm, vias 384 -> 385

Commit message: GND repair: island bridging + per-pad vias before routing; nodemcu manufacturing files
Co-Authored-By: Claude Fable 5.1 <noreply@anthropic.com>
Claude-Session: https://claude.ai/code/session_01BYqUw5RUauFb8joYQgSgKZ
Routing:
- net GND: track 11.6 -> 18.6 mm, vias 385 -> 390

Commit message: Module variant: routed, DRC-clean board and manufacturing files; net-level reroute tool
Co-Authored-By: Claude Fable 5.1 <noreply@anthropic.com>
Claude-Session: https://claude.ai/code/session_01BYqUw5RUauFb8joYQgSgKZ
Routing:
- net GND: track 18.6 -> 11.6 mm, vias 390 -> 385
