File: openchess-redesign/hardware-nodemcu/openchess-board-nodemcu.kicad_pcb (KiCad board)
At the start: 2 copper layers, 340 x 388 mm, 239 parts, among them J1 USB-C, J2 5V IN, J3 DEV_TOP, J4 DEV_BOTTOM, Q1 S8550, Q2 S8550, Q3 S8550, Q4 S8550, Q5 S8550, Q6 S8550, Q7 S8550, Q8 S8550, U4 74HCT595, U5 74AHCT1G125

Commit message: NodeMCU variant: routed, DRC-clean board and manufacturing files
build.sh: default 12 router passes (30 passes can loop on this strip).

Co-Authored-By: Claude Fable 5.1 <noreply@anthropic.com>
Claude-Session: https://claude.ai/code/session_01BYqUw5RUauFb8joYQgSgKZ
Routing:
- net +3V3: track 0.00 -> 165.6 mm, vias 0 -> 2
- net IO33: track 0.00 -> 161.5 mm, vias 0 -> 1
- net IO26: track 0.00 -> 153.5 mm, vias 0 -> 1
- net IO14: track 0.00 -> 144.6 mm, vias 0 -> 1
- net +5V: track 3418.4 -> 3549.9 mm, vias 75 -> 80
- net ROW7: track 626.9 -> 683.1 mm, vias 1 -> 3
- net ROW3: track 470.1 -> 525.1 mm, vias 1 -> 4
- net ROW1: track 391.7 -> 445.5 mm, vias 1 -> 4
- net IO32: track 0.00 -> 51.0 mm
- net ROW2: track 430.9 -> 478.2 mm, vias 1 -> 5
- net ROW5: track 548.5 -> 594.2 mm, vias 1 -> 4
- net ROW6: track 587.7 -> 630.7 mm, vias 1 -> 4
- net ROW0: track 352.5 -> 395.4 mm
- net SRQ3: track 17.8 -> 59.8 mm, vias 0 -> 2
- net SRQ4: track 3.93 -> 42.4 mm, vias 0 -> 2
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
Commit message: Add optional IP5306 battery charger/boost block with power-select jumper
Fuse -> JP1 pin 1 / IP5306 VIN; IP5306 VOUT -> JP1 pin 3; JP1 pin 2 -> 5V bus.
JST-PH battery connector, key button, 1 uH inductor, 3x 22 uF. Wide power
paths pre-routed; enclosure cover gets openings for J5, SW3 and JP1.

Co-Authored-By: Claude Fable 5.1 <noreply@anthropic.com>
Claude-Session: https://claude.ai/code/session_01BYqUw5RUauFb8joYQgSgKZ
Parts:
- added C77: 22uF, Capacitor_SMD:C_0805_2012Metric, F.Cu at (226.3, 366.5)
- added C78: 22uF, Capacitor_SMD:C_0805_2012Metric, F.Cu at (252.0, 372.5)
- added C79: 22uF, Capacitor_SMD:C_0805_2012Metric, F.Cu at (242.0, 365.0)
- added J5: BATTERY, Connector_JST:JST_PH_B2B-PH-K_1x02_P2.00mm_Vertical, F.Cu at (262.0, 383.0)
- added JP1: PWR SEL, Connector_PinHeader_2.54mm:PinHeader_1x03_P2.54mm_Vertical, F.Cu at (193.5, 379.5)
- added L1: 1uH 4A, Inductor_SMD:L_Taiyo-Yuden_NR-60xx, F.Cu at (242.0, 371.4)
- added SW3: PWR, Button_Switch_SMD:SW_SPST_TL3342, F.Cu at (276.0, 382.0)
- added U6: IP5306, Package_SO:HSOP-8-1EP_3.9x4.9mm_P1.27mm_EP2.41x3.1mm_ThermalVias, F.Cu at (232.0, 372.0)
Connections:
- F1 pad 2: +5V -> VUSB5
Routing:
- net VUSB5: track 0.00 -> 165.9 mm
- net +3V3: track 165.6 -> 0.00 mm, vias 2 -> 0
- net IO33: track 161.5 -> 0.00 mm, vias 1 -> 0
- net IO26: track 153.5 -> 0.00 mm, vias 1 -> 0
- net IO14: track 144.6 -> 0.00 mm, vias 1 -> 0
- net +5V: track 3549.9 -> 3441.9 mm, vias 80 -> 72
- net VBOOST: track 0.00 -> 69.4 mm
- net ROW7: track 683.1 -> 626.9 mm, vias 3 -> 1
- net ROW3: track 525.1 -> 470.1 mm, vias 4 -> 1
- net ROW1: track 445.5 -> 391.7 mm, vias 4 -> 1
- net IO32: track 51.0 -> 0.00 mm
- net ROW2: track 478.2 -> 430.9 mm, vias 5 -> 1
- net ROW5: track 594.2 -> 548.5 mm, vias 4 -> 1
- net BAT: track 0.00 -> 43.8 mm
- net ROW6: track 630.7 -> 587.7 mm, vias 4 -> 1
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Other:
- board text added: "BAT 1S Li-ion + left"
- board text added: "J1 USB-C 5V/3A | J2 5V/4A in"
- board text added: "JP1: 1-2 USB 2-3 BATTERY"
- board text added: "LED IO32 | SER IO33 SRCLK IO14 RCLK IO26"
- board text added: "OpenChess PCB v1.0 (nodemcu)"
- board text added: "ROW1..8 = IO4,16,17,18,19,21,22,23"
- board text added: "SR_INVERT_OUTPUTS = PNP (WebUI)"
- board text removed: "Column drivers are PNP: set SR_INVERT_OUTPUTS = PNP in the WebUI. J1 USB-C 5V/3A (fused) | J2 ext 5V 4A"
- board text removed: "GPIO: LED IO32 | SR SER IO33 SRCLK IO14 RCLK IO26 | ROW1..8 = IO4,16,17,18,19,21,22,23"
- board text removed: "OpenChess PCB redesign v1.0 (nodemcu) - 8x8 Hall + WS2812B, firmware-compatible with joojoooo/OpenChess"

Commit message: Both variants routed and DRC-clean with the battery block; manufacturing files and enclosure STLs regenerated
Co-Authored-By: Claude Fable 5.1 <noreply@anthropic.com>
Claude-Session: https://claude.ai/code/session_01BYqUw5RUauFb8joYQgSgKZ
Routing:
- net +5V: track 3441.9 -> 3607.9 mm, vias 72 -> 75
- net +3V3: track 0.00 -> 165.0 mm, vias 0 -> 2
- net IO33: track 0.00 -> 164.2 mm, vias 0 -> 1
- net IO14: track 0.00 -> 162.7 mm, vias 0 -> 2
- net IO26: track 0.00 -> 155.7 mm, vias 0 -> 1
- net IO32: track 0.00 -> 59.2 mm, vias 0 -> 2
- net ROW7: track 626.9 -> 684.1 mm, vias 1 -> 3
- net KEY: track 0.00 -> 51.3 mm
- net ROW3: track 470.1 -> 520.5 mm, vias 1 -> 4
- net ROW1: track 391.7 -> 441.0 mm, vias 1 -> 3
- net ROW2: track 430.9 -> 478.4 mm
- net ROW0: track 352.5 -> 399.0 mm, vias 1 -> 2
- net ROW6: track 587.7 -> 631.2 mm, vias 1 -> 2
- net ROW4: track 509.3 -> 551.3 mm, vias 1 -> 2
- net ROW5: track 548.5 -> 589.7 mm, vias 1 -> 2
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