File: openchess-redesign/hardware/openchess-board.kicad_pcb (KiCad board)
At the start: 2 copper layers, 340 x 374 mm, 255 parts, among them J1 USB-C, J2 5V IN, Q1 S8550, Q10 S8050, Q2 S8550, Q3 S8550, Q4 S8550, Q5 S8550, Q6 S8550, Q7 S8550, Q8 S8550, Q9 S8050, SW1 RESET, SW2 BOOT, U1 ESP32-WROOM-32E, U2 AMS1117-3.3, U3 CH340C, U4 74HCT595, U5 74AHCT1G125

Commit message: Pre-route USB-C escape and VBUS, stitch strip ground, add SES importer
KiCad 7 cannot import a Specctra session headless, so tools/ses_import.py
reads the Freerouting .ses directly. Also trims bus ends, cleans dangling
autorouter tails and solid-connects USB-C GND pads to the pour.

Co-Authored-By: Claude Fable 5.1 <noreply@anthropic.com>
Claude-Session: https://claude.ai/code/session_01BYqUw5RUauFb8joYQgSgKZ
Parts:
- moved R18 8.06 mm to (87.0, 366.0)
- moved R17 7.21 mm to (70.0, 366.0)
- moved U3 2.00 mm to (78.0, 352.0)
- moved C71 1.00 mm to (70.0, 348.0)
- moved C72 1.00 mm to (86.0, 348.0)
Routing:
- net USB_D+: track 0.00 -> 21.9 mm
- net USB_D-: track 0.00 -> 20.0 mm, vias 0 -> 2
- net +5V: track 3410.3 -> 3394.4 mm
- net CC1: track 0.00 -> 7.25 mm
- net CC2: track 0.00 -> 6.69 mm
- net VBUS: track 26.9 -> 33.3 mm, vias 0 -> 3
- net GND: vias 115 -> 332
- net CH_V3: vias 0 -> 1

Commit message: Add GND island repair, router clearance margin, T-junction-aware tail cleanup
Co-Authored-By: Claude Fable 5.1 <noreply@anthropic.com>
Claude-Session: https://claude.ai/code/session_01BYqUw5RUauFb8joYQgSgKZ
Parts:
- moved J2 10.0 mm to (118.0, 369.0)
Routing:
- net +5V: track 3394.4 -> 3404.4 mm
- net GND: vias 332 -> 289
Other:
- board text added: "OpenChess PCB redesign v1.0 (module) - 8x8 Hall + WS2812B, firmware-compatible with joojoooo/OpenChess"
- board text removed: "OpenChess PCB redesign v1.0 - 8x8 Hall + WS2812B, firmware-compatible with joojoooo/OpenChess"

Commit message: Pre-route 74HCT595 OE ground via; router margin 0.02 mm; GND repair adds pad stubs
Co-Authored-By: Claude Fable 5.1 <noreply@anthropic.com>
Claude-Session: https://claude.ai/code/session_01BYqUw5RUauFb8joYQgSgKZ
Routing:
- net GND: track 0.00 -> 2.60 mm, vias 289 -> 290

Commit message: GND repair: island bridging + per-pad vias before routing; nodemcu manufacturing files
Co-Authored-By: Claude Fable 5.1 <noreply@anthropic.com>
Claude-Session: https://claude.ai/code/session_01BYqUw5RUauFb8joYQgSgKZ
Routing:
- net GND: track 2.60 -> 19.4 mm, vias 290 -> 301

Commit message: module: pre-route ESP32 GND pins to the thermal pad; repair uses exact track distances
Co-Authored-By: Claude Fable 5.1 <noreply@anthropic.com>
Claude-Session: https://claude.ai/code/session_01BYqUw5RUauFb8joYQgSgKZ
Routing:
- net GND: track 19.4 -> 77.7 mm

Commit message: Module variant: routed, DRC-clean board and manufacturing files; net-level reroute tool
Co-Authored-By: Claude Fable 5.1 <noreply@anthropic.com>
Claude-Session: https://claude.ai/code/session_01BYqUw5RUauFb8joYQgSgKZ
Routing:
- net +3V3: track 0.00 -> 172.2 mm, vias 0 -> 4
- net IO26: track 0.00 -> 164.5 mm, vias 0 -> 2
- net IO14: track 0.00 -> 160.9 mm, vias 0 -> 4
- net IO33: track 0.00 -> 153.1 mm, vias 0 -> 2
- net ROW3: track 461.1 -> 576.9 mm, vias 1 -> 3
- net +5V: track 3404.4 -> 3506.1 mm, vias 75 -> 79
- net SRQ0: track 140.2 -> 240.2 mm, vias 0 -> 2
- net ROW7: track 617.9 -> 703.9 mm, vias 1 -> 3
- net IO0: track 0.00 -> 84.2 mm, vias 0 -> 2
- net ROW6: track 578.7 -> 655.3 mm, vias 1 -> 4
- net TXD0: track 0.00 -> 76.1 mm, vias 0 -> 2
- net RXD0: track 0.00 -> 72.3 mm, vias 0 -> 2
- net EN: track 0.00 -> 72.0 mm, vias 0 -> 2
- net ROW4: track 500.3 -> 568.3 mm, vias 1 -> 3
- net ROW1: track 382.7 -> 442.5 mm, vias 1 -> 5
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
Commit message: Add optional IP5306 battery charger/boost block with power-select jumper
Fuse -> JP1 pin 1 / IP5306 VIN; IP5306 VOUT -> JP1 pin 3; JP1 pin 2 -> 5V bus.
JST-PH battery connector, key button, 1 uH inductor, 3x 22 uF. Wide power
paths pre-routed; enclosure cover gets openings for J5, SW3 and JP1.

Co-Authored-By: Claude Fable 5.1 <noreply@anthropic.com>
Claude-Session: https://claude.ai/code/session_01BYqUw5RUauFb8joYQgSgKZ
Parts:
- added C77: 22uF, Capacitor_SMD:C_0805_2012Metric, F.Cu at (226.3, 352.5)
- added C78: 22uF, Capacitor_SMD:C_0805_2012Metric, F.Cu at (252.0, 358.5)
- added C79: 22uF, Capacitor_SMD:C_0805_2012Metric, F.Cu at (242.0, 351.0)
- added J5: BATTERY, Connector_JST:JST_PH_B2B-PH-K_1x02_P2.00mm_Vertical, F.Cu at (262.0, 369.0)
- added JP1: PWR SEL, Connector_PinHeader_2.54mm:PinHeader_1x03_P2.54mm_Vertical, F.Cu at (193.5, 365.5)
- added L1: 1uH 4A, Inductor_SMD:L_Taiyo-Yuden_NR-60xx, F.Cu at (242.0, 357.4)
- added SW3: PWR, Button_Switch_SMD:SW_SPST_TL3342, F.Cu at (276.0, 368.0)
- added U6: IP5306, Package_SO:HSOP-8-1EP_3.9x4.9mm_P1.27mm_EP2.41x3.1mm_ThermalVias, F.Cu at (232.0, 358.0)
Connections:
- F1 pad 2: +5V -> VUSB5
Routing:
- net +3V3: track 172.2 -> 0.00 mm, vias 4 -> 0
- net VUSB5: track 0.00 -> 165.9 mm
- net IO26: track 164.5 -> 0.00 mm, vias 2 -> 0
- net IO14: track 160.9 -> 0.00 mm, vias 4 -> 0
- net IO33: track 153.1 -> 0.00 mm, vias 2 -> 0
- net ROW3: track 576.9 -> 461.1 mm, vias 3 -> 1
- net SRQ0: track 240.2 -> 140.2 mm, vias 2 -> 0
- net +5V: track 3506.1 -> 3413.9 mm, vias 79 -> 72
- net ROW7: track 703.9 -> 617.9 mm, vias 3 -> 1
- net IO0: track 84.2 -> 0.00 mm, vias 2 -> 0
- net ROW6: track 655.3 -> 578.7 mm, vias 4 -> 1
- net TXD0: track 76.1 -> 0.00 mm, vias 2 -> 0
- net RXD0: track 72.3 -> 0.00 mm, vias 2 -> 0
- net EN: track 72.0 -> 0.00 mm, vias 2 -> 0
- net VBOOST: track 0.00 -> 69.4 mm, vias 0 -> 1
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Other:
- board text added: "BAT 1S Li-ion + left"
- board text added: "J1 USB-C 5V/3A | J2 5V/4A in"
- board text added: "JP1: 1-2 USB 2-3 BATTERY"
- board text added: "LED IO32 | SER IO33 SRCLK IO14 RCLK IO26"
- board text added: "OpenChess PCB v1.0 (module)"
- board text added: "ROW1..8 = IO4,16,17,18,19,21,22,23"
- board text added: "SR_INVERT_OUTPUTS = PNP (WebUI)"
- board text removed: "Column drivers are PNP: set SR_INVERT_OUTPUTS = PNP in the WebUI. J1 USB-C 5V/3A (fused) | J2 ext 5V 4A"
- board text removed: "GPIO: LED IO32 | SR SER IO33 SRCLK IO14 RCLK IO26 | ROW1..8 = IO4,16,17,18,19,21,22,23"
- board text removed: "OpenChess PCB redesign v1.0 (module) - 8x8 Hall + WS2812B, firmware-compatible with joojoooo/OpenChess"

Commit message: Both variants routed and DRC-clean with the battery block; manufacturing files and enclosure STLs regenerated
Co-Authored-By: Claude Fable 5.1 <noreply@anthropic.com>
Claude-Session: https://claude.ai/code/session_01BYqUw5RUauFb8joYQgSgKZ
Routing:
- net ROW6: track 578.7 -> 805.8 mm, vias 1 -> 4
- net IO14: track 0.00 -> 178.4 mm, vias 0 -> 2
- net IO33: track 0.00 -> 167.8 mm, vias 0 -> 2
- net IO26: track 0.00 -> 164.4 mm, vias 0 -> 6
- net +3V3: track 0.00 -> 159.8 mm, vias 0 -> 4
- net +5V: track 3413.9 -> 3570.2 mm, vias 72 -> 74
- net IO0: track 0.00 -> 95.4 mm, vias 0 -> 3
- net ROW4: track 500.3 -> 593.3 mm, vias 1 -> 6
- net ROW7: track 617.9 -> 692.8 mm, vias 1 -> 3
- net TXD0: track 0.00 -> 74.1 mm, vias 0 -> 2
- net RXD0: track 0.00 -> 72.0 mm, vias 0 -> 2
- net EN: track 0.00 -> 71.3 mm, vias 0 -> 2
- net ROW5: track 539.5 -> 609.4 mm, vias 1 -> 5
- net ROW3: track 461.1 -> 524.8 mm, vias 1 -> 3
- net SRQ0: track 140.2 -> 199.8 mm, vias 0 -> 2
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