File: openchess-redesign/hardware/openchess-board.kicad_sch (KiCad schematic)
At the start: 255 parts, among them J1 USB-C, J2 5V IN, Q1 S8550, Q10 S8050, Q2 S8550, Q3 S8550, Q4 S8550, Q5 S8550, Q6 S8550, Q7 S8550, Q8 S8550, Q9 S8050, SW1 RESET, SW2 BOOT, U1 ESP32-WROOM-32E, U2 AMS1117-3.3, U3 CH340C, U4 74HCT595, U5 74AHCT1G125

Commit message: Add optional IP5306 battery charger/boost block with power-select jumper
Fuse -> JP1 pin 1 / IP5306 VIN; IP5306 VOUT -> JP1 pin 3; JP1 pin 2 -> 5V bus.
JST-PH battery connector, key button, 1 uH inductor, 3x 22 uF. Wide power
paths pre-routed; enclosure cover gets openings for J5, SW3 and JP1.

Co-Authored-By: Claude Fable 5.1 <noreply@anthropic.com>
Claude-Session: https://claude.ai/code/session_01BYqUw5RUauFb8joYQgSgKZ
Parts:
- added C77, C78, C79: 22uF, Capacitor_SMD:C_0805_2012Metric, symbol Device:C
- added J5: BATTERY, Connector_JST:JST_PH_B2B-PH-K_1x02_P2.00mm_Vertical, symbol Connector_Generic:Conn_01x02
- added JP1: PWR SEL, Connector_PinHeader_2.54mm:PinHeader_1x03_P2.54mm_Vertical, symbol Connector_Generic:Conn_01x03
- added L1: 1uH 4A, Inductor_SMD:L_Taiyo-Yuden_NR-60xx, symbol Device:L
- added SW3: PWR, Button_Switch_SMD:SW_SPST_TL3342, symbol Switch:SW_Push
- added U6: IP5306, Package_SO:HSOP-8-1EP_3.9x4.9mm_P1.27mm_EP2.41x3.1mm_ThermalVias, symbol OpenChess:IP5306
Connections:
- net +5V: now also JP1.2 (Pin_2); no longer F1.2
- net GND: now also C77.2, C78.2, C79.2, J5.2 (Pin_2), SW3.2, U6.9 (GND)
- new net BAT: C78.1, J5.1 (Pin_1), L1.2, U6.6 (BAT)
- new net KEY: SW3.1, U6.5 (KEY)
- new net LX: L1.1, U6.7 (L1)
- new net VBOOST: C79.1, JP1.3 (Pin_3), U6.8 (VOUT)
- new net VUSB5: C77.1, F1.2, JP1.1 (Pin_1), U6.1 (VIN)
- no-connect marks 29 -> 32
Other:
- note added: "OPTIONAL BATTERY: IP5306 charges a 1S Li-ion from VUSB5 and boosts it to 5 V. JP1 1-2 = USB direct, 2-3 = battery/boost."
- title: OpenChess PCB redesign - 8x8 Hall/WS2812B board -> OpenChess PCB redesign - 8x8 Hall/WS2812B board (module variant)

Commit message: Pre-order checklist: confirmed LCSC numbers, fixed PNP/NPN part numbers, no-battery BOM/CPL variants
Co-Authored-By: Claude Fable 5.1 <noreply@anthropic.com>
Claude-Session: https://claude.ai/code/session_01BYqUw5RUauFb8joYQgSgKZ
Parts:
- C75, C76: LCSC (none) -> C3341; MPN 470uF/10V SMD 8x10 -> RVT1C471M0810 470uF 16V D8xL10 (verify)
- F1: LCSC (none) -> C883162; MPN MF-MSMF300-2 / BSMD1812-300 -> BSMD1812-300-16V (BHFUSE) or ASMD1812-300 C135366
- H1, H10, H11, H12, H13, H14, H15, H16, H17, H18, H19, H2, H20, H21, H22, H23, H24, H25, H26, H27, H28, H29, H3, H30, H31, H32, H33, H34, H35, H36, H37, H38, H39, H4, H40, H41, H42, H43, H44, H45, H46, H47, H48, H49, H5, H50, H51, H52, H53, H54, H55, H56, H57, H58, H59, H6, H60, H61, H62, H63, H64, H7, H8, H9: LCSC (none) -> C558880
- JP1: LCSC C2337 -> (none); MPN 1x3 header + jumper -> 1x3 pin header 2.54 mm + jumper cap
- L1: LCSC (none) -> C96955; MPN NR6028T1R0N / CD63 1uH >=4A -> SWPA6045S1R0NT (Sunlord) / CKCS6045-1uH/N C354627 / NR6045T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
- Q1, Q2, Q3, Q4, Q5, Q6, Q7, Q8: LCSC C2150 -> C2147; MPN S8550 -> S8550 2TY (PNP)
- Q10, Q9: MPN S8050 -> S8050 J3Y (NPN)
- R23: MPN (none) -> 330R 0603 (verify C23138)
- U4: LCSC (none) -> C70468; MPN SN74HCT595DR / 74HCT595D -> 74HCT595D,112 (Nexperia)
- U5: LCSC (none) -> C7484
